File: kicad/rpi-atmega324-modbus-x3-gateway.kicad_pcb (KiCad board)
At the start: 4 copper layers, 84.2 x 86.3 mm, 142 parts, among them J1 Raspberry_Pi_2+, J10 Conn_01x03, J11 SOLDERBRDIGE-3, J12 Conn_01x02, J13 Conn_01x02, J14 Conn_01x02, J15 SOLDERBRDIGE-2, J16 Screw_Terminal_01x02, J17 PRJ_USB_MINI, J18 Conn_01x05, J19 SOLDERBRDIGE-3, J2 UART-Harwin3, J20 Conn_01x05, J21 SOLDERBRDIGE-3, J22 SOLDERBRDIGE-2, J23 UART-Harwin3, J24 Conn_02x03_Odd_Even, J25 Atmega-ISP-6, J26 Conn_01x03, J27 Conn_01x03, J28 Conn_01x02, J29 Conn_01x02, J3 Conn_01x04, J30 Conn_01x02, J31 Conn_01x02, J32 Conn_01x02, J33 Conn_01x02, J34 Conn_01x04, J35 Screw_Terminal_01x02, J36 Screw_Terminal_01x02, J37 Screw_Terminal_01x03, J38 Conn_01x02, J39 Conn_01x02, J4 Conn_01x04, J5 SOLDERBRDIGE-3, J6 Conn_02x03_Odd_Even, J7 Conn_01x05, J8 Atmega-ISP-6, J9 PRJ_USB_MINI, SW1 SW_Push, SW2 SW_Push, U1 PRJ-UC1-ATMEGA324P-20AU, U2 PRJ-UC2-ATMEGA324P-20AU, U3 SN65HVD11, U4 CH340G, U5 CH340G, U6 SN65HVD11, U7 SN65HVD11, U8 HLK-5M05, Y1 12MHz, Y2 12MHz, Y3 12MHz, Y4 12MHz

Commit message: PCB V0.1 Tapeout
Parts:
- moved R32 12.5 mm to (148.9, 117.1), turned to 90 degrees
- moved J4 1.63 mm to (122.3, 72.9)
- moved C16 1.30 mm to (157.9, 111.8)
- moved R33 0.89 mm to (157.5, 109.6)
- moved D3 0.83 mm to (121.9, 132.5)
- moved D4 0.83 mm to (109.2, 132.5)
- moved R36 0.81 mm to (146.5, 122.4)
- moved D20 0.81 mm to (126.5, 132.5)
- moved D14 0.81 mm to (160.3, 132.5)
- moved D15 0.81 mm to (147.6, 132.5)
- moved D19 0.81 mm to (139.2, 132.5)
- moved R9 0.64 mm to (109.0, 129.2)
- moved Y3 0.60 mm to (156.1, 67.4)
- moved R5 0.51 mm to (122.0, 129.3)
- moved J23 0.51 mm to (177.8, 77.5)
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Connections:
- net Net-(J10-Pad2) renamed /uc1/B1-A
- net Net-(J10-Pad3) renamed /uc1/B1-B
- net Net-(J26-Pad2) renamed /uc2/B3-A
- net Net-(J26-Pad3) renamed /uc2/B3-B
- net Net-(J27-Pad2) renamed /uc2/B2-A
- net Net-(J27-Pad3) renamed /uc2/B2-B
Routing:
- net /uc2/B3-A: track 21.4 -> 37.7 mm
- net /uc2/Modbus3-A: track 54.8 -> 39.5 mm
- net GND: track 147.9 -> 160.7 mm
- net /uc1/MODBUS1-DE: track 63.2 -> 69.8 mm, vias 6 -> 7
- net /uc2/UC2-TxD0: track 130.8 -> 128.0 mm
- net Net-(D5-Pad2): track 3.63 -> 6.05 mm
- net /uc2/USB2-RxD: track 14.3 -> 12.1 mm
- net Net-(J24-Pad4): track 76.2 -> 74.1 mm
- net /uc1/UC1-RxD1: track 82.5 -> 80.5 mm
- net Net-(C8-Pad1): track 9.00 -> 7.37 mm
- net Net-(U4-Pad8): track 8.90 -> 10.4 mm
- net Net-(D6-Pad2): track 3.63 -> 5.11 mm
- net Net-(D14-Pad1): track 25.9 -> 27.3 mm
- net /uc1/~RESET~: track 79.7 -> 78.4 mm
- net /uc1/UC1-PA1: track 16.7 -> 15.5 mm
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Other:
- board text added: "B1"
- board text added: "B3"
- board text added: "DE"
- board text added: "GND"
- board text added: "GND A B"
- board text added: "N-230V-L"
- board text added: "PA0"
- board text added: "PA1"
- board text added: "PA2"
- board text added: "PC3"
- board text added: "PC4"
- board text added: "PC5"
- board text added: "PD"
- board text added: "PU"
- board text added: "Rx"
- board text added: "Rx0"
- board text added: "TERM"
- board text added: "Tx"
- board text added: "Tx0"
- board text added: "Version"
- board text added: "~CS~"
- board text added: "~RE~"
- board text removed: "N 230V L"
