File: kicad/uc1.sch (KiCad schematic (older format))
At the start: 58 parts, among them J10 Conn_01x03, J11 SOLDERBRDIGE-3, J12 Conn_01x02, J13 Conn_01x02, J14 Conn_01x02, J15 SOLDERBRDIGE-2, J16 Screw_Terminal_01x02, J2 UART-Harwin3, J3 Conn_01x04, J38 Conn_01x02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

Commit message: PCB V0.1 Tapeout
Connections:
- net labels added: B1-A, B1-B
Changed lines of the file:
@@
 $EndDescr
 $Comp
-L +3.3V #PWR14
+L +3.3V #PWR09
 U 1 1 5B8BF8F1
 P 3900 1000
-F 0 "#PWR14" H 3900 850 50  0001 C CNN
+F 0 "#PWR09" H 3900 850 50  0001 C CNN
 F 1 "+3.3V" H 3900 1140 50  0000 C CNN
 F 2 "" H 3900 1000 50  0001 C CNN
@@
 $EndComp
 $Comp
-L GND #PWR15
+L GND #PWR010
 U 1 1 5B8BF95B
 P 3900 5800
-F 0 "#PWR15" H 3900 5550 50  0001 C CNN
+F 0 "#PWR010" H 3900 5550 50  0001 C CNN
 F 1 "GND" H 3900 5650 50  0000 C CNN
 F 2 "" H 3900 5800 50  0001 C CNN
@@
 $EndComp
 $Comp
-L GND #PWR16
+L GND #PWR011
 U 1 1 5B8C015E
 P 5000 1600
-F 0 "#PWR16" H 5000 1350 50  0001 C CNN
+F 0 "#PWR011" H 5000 1350 50  0001 C CNN
 F 1 "GND" H 5000 1450 50  0000 C CNN
 F 2 "" H 5000 1600 50  0001 C CNN
@@
 $EndComp
 $Comp
-L GND #PWR13
+L GND #PWR012
 U 1 1 5B8C042C
 P 3000 3700
-F 0 "#PWR13" H 3000 3450 50  0001 C CNN
+F 0 "#PWR012" H 3000 3450 50  0001 C CNN
 F 1 "GND" H 3000 3550 50  0000 C CNN
 F 2 "" H 3000 3700 50  0001 C CNN
@@
 	3000 3700 3000 3650
 $Comp
-L GND #PWR9
+L GND #PWR013
 U 1 1 5B8C078E
 P 2100 3000
-F 0 "#PWR9" H 2100 2750 50  0001 C CNN
+F 0 "#PWR013" H 2100 2750 50  0001 C CNN
 F 1 "GND" H 2100 2850 50  0000 C CNN
 F 2 "" H 2100 3000 50  0001 C CNN
@@
 Connection ~ 2300 4100
 $Comp
-L +3.3V #PWR10
+L +3.3V #PWR014
 U 1 1 5B8C232B
 P 2300 3600
-F 0 "#PWR10" H 2300 3450 50  0001 C CNN
+F 0 "#PWR014" H 2300 3450 50  0001 C CNN
 F 1 "+3.3V" H 2300 3740 50  0000 C CNN
 F 2 "" H 2300 3600 50  0001 C CNN
@@
 $EndComp
 $Comp
-L +3.3V #PWR11
+L +3.3V #PWR015
 U 1 1 5B8CF934
 P 2600 800
-F 0 "#PWR11" H 2600 650 50  0001 C CNN
+F 0 "#PWR015" H 2600 650 50  0001 C CNN
 F 1 "+3.3V" H 2600 940 50  0000 C CNN
 F 2 "" H 2600 800 50  0001 C CNN
@@
 $EndComp
 $Comp
-L GND #PWR8
+L GND #PWR016
 U 1 1 5B8CFAF7
 P 1900 2100
-F 0 "#PWR8" H 1900 1850 50  0001 C CNN
+F 0 "#PWR016" H 1900 1850 50  0001 C CNN
 F 1 "GND" H 1900 1950 50  0000 C CNN
 F 2 "" H 1900 2100 50  0001 C CNN
@@
 $EndComp
 $Comp
-L +3.3V #PWR34
+L +3.3V #PWR017
 U 1 1 5B8D4C88
 P 9500 900
-F 0 "#PWR34" H 9500 750 50  0001 C CNN
+F 0 "#PWR017" H 9500 750 50  0001 C CNN
 F 1 "+3.3V" H 9500 1040 50  0000 C CNN
 F 2 "" H 9500 900 50  0001 C CNN
@@
 	9800 2800 9800 2700
 $Comp
-L GND #PWR37
+L GND #PWR018
 U 1 1 5B8D4F3C
 P 10100 2400
-F 0 "#PWR37" H 10100 2150 50  0001 C CNN
+F 0 "#PWR018" H 10100 2150 50  0001 C CNN
 F 1 "GND" H 10100 2250 50  0000 C CNN
 F 2 "" H 10100 2400 50  0001 C CNN
@@
 	9500 3200 9500 3300
 $Comp
-L GND #PWR35
+L GND #PWR019
 U 1 1 5B8D63D4
 P 9500 3700
-F 0 "#PWR35" H 9500 3450 50  0001 C CNN
+F 0 "#PWR019" H 9500 3450 50  0001 C CNN
 F 1 "GND" H 9500 3550 50  0000 C CNN
 F 2 "" H 9500 3700 50  0001 C CNN
@@
 	8000 2200 8000 1500
 $Comp
-L GND #PWR30
+L GND #PWR020
 U 1 1 5B8D844E
 P 7900 1700
-F 0 "#PWR30" H 7900 1450 50  0001 C CNN
+F 0 "#PWR020" H 7900 1450 50  0001 C CNN
 F 1 "GND" H 7900 1550 50  0000 C CNN
 F 2 "" H 7900 1700 50  0001 C CNN
@@
 $EndComp
 $Comp
-L GND #PWR24
+L GND #PWR021
 U 1 1 5B8DC717
 P 6700 3100
-F 0 "#PWR24" H 6700 2850 50  0001 C CNN
+F 0 "#PWR021" H 6700 2850 50  0001 C CNN
 F 1 "GND" H 6700 2950 50  0000 C CNN
 F 2 "" H 6700 3100 50  0001 C CNN
@@
 Connection ~ 6500 2500
 $Comp
-L +3.3V #PWR23
+L +3.3V #PWR022
 U 1 1 5B8DCB13
 P 6600 1500
-F 0 "#PWR23" H 6600 1350 50  0001 C CNN
+F 0 "#PWR022" H 6600 1350 50  0001 C CNN
 F 1 "+3.3V" H 6600 1640 50  0000 C CNN
 F 2 "" H 6600 1500 50  0001 C CNN
@@
 $EndComp
 $Comp
-L +3.3V #PWR18
+L +3.3V #PWR023
 U 1 1 5B8DD67E
 P 6000 1100
-F 0 "#PWR18" H 6000 950 50  0001 C CNN
+F 0 "#PWR023" H 6000 950 50  0001 C CNN
 F 1 "+3.3V" H 6000 1240 50  0000 C CNN
 F 2 "" H 6000 1100 50  0001 C CNN
@@
 Connection ~ 6100 2500
 $Comp
-L +3.3V #PWR26
+L +3.3V #PWR024
 U 1 1 5B8DDB3F
 P 7300 1400
-F 0 "#PWR26" H 7300 1250 50  0001 C CNN
+F 0 "#PWR024" H 7300 1250 50  0001 C CNN
 F 1 "+3.3V" H 7300 1540 50  0000 C CNN
 F 2 "" H 7300 1400 50  0001 C CNN
@@
 Connection ~ 7900 1600
 $Comp
-L GND #PWR27
+L GND #PWR025
 U 1 1 5B8DE192
 P 7300 3000
-F 0 "#PWR27" H 7300 2750 50  0001 C CNN
+F 0 "#PWR025" H 7300 2750 50  0001 C CNN
 F 1 "GND" H 7300 2850 50  0000 C CNN
 F 2 "" H 7300 3000 50  0001 C CNN
@@
 $EndComp
 $Comp
-L GND #PWR32
+L GND #PWR026
 U 1 1 5B8E1773
 P 8500 5900
-F 0 "#PWR32" H 8500 5650 50  0001 C CNN
+F 0 "#PWR026" H 8500 5650 50  0001 C CNN
 F 1 "GND" H 8500 5750 50  0000 C CNN
 F 2 "" H 8500 5900 50  0001 C CNN
@@
 $EndComp
 $Comp
-L GND #PWR29
+L GND #PWR027
 U 1 1 5B8E17F3
 P 7700 5400
-F 0 "#PWR29" H 7700 5150 50  0001 C CNN
+F 0 "#PWR027" H 7700 5150 50  0001 C CNN
 F 1 "GND" H 7700 5250 50  0000 C CNN
 F 2 "" H 7700 5400 50  0001 C CNN
@@
 	8500 5800 8500 5900
 $Comp
-L +3.3V #PWR33
+L +3.3V #PWR028
 U 1 1 5B8E1DF2
 P 9100 3600
-F 0 "#PWR33" H 9100 3450 50  0001 C CNN
+F 0 "#PWR028" H 9100 3450 50  0001 C CNN
 F 1 "+3.3V" H 9100 3740 50  0000 C CNN
 F 2 "" H 9100 3600 50  0001 C CNN
@@
 	8200 4800 7300 4800
 $Comp
-L GND #PWR25
+L GND #PWR029
 U 1 1 5B8E2C87
 P 7000 5300
-F 0 "#PWR25" H 7000 5050 50  0001 C CNN
+F 0 "#PWR029" H 7000 5050 50  0001 C CNN
 F 1 "GND" H 7000 5150 50  0000 C CNN
 F 2 "" H 7000 5300 50  0001 C CNN
@@
 $EndComp
 $Comp
-L GND #PWR31
+L GND #PWR030
 U 1 1 5B8E3267
 P 8000 4300
-F 0 "#PWR31" H 8000 4050 50  0001 C CNN
+F 0 "#PWR030" H 8000 4050 50  0001 C CNN
 F 1 "GND" H 8000 4150 50  0000 C CNN
 F 2 "" H 8000 4300 50  0001 C CNN
@@
 UC1-MOSI
 $Comp
-L GND #PWR22
+L GND #PWR031
 U 1 1 5B8E5FA1
 P 6100 6800
-F 0 "#PWR22" H 6100 6550 50  0001 C CNN
+F 0 "#PWR031" H 6100 6550 50  0001 C CNN
 F 1 "GND" H 6100 6650 50  0000 C CNN
 F 2 "" H 6100 6800 50  0001 C CNN
@@
 	6100 6600 6100 6800
 $Comp
-L +3.3V #PWR21
+L +3.3V #PWR032
 U 1 1 5B8E616A
 P 6100 6200
-F 0 "#PWR21" H 6100 6050 50  0001 C CNN
+F 0 "#PWR032" H 6100 6050 50  0001 C CNN
 F 1 "+3.3V" H 6100 6340 50  0000 C CNN
 F 2 "" H 6100 6200 50  0001 C CNN
@@
 $EndComp
 $Comp
-L +3.3V #PWR12
+L +3.3V #PWR033
 U 1 1 5B8D98CD
 P 2800 5200
-F 0 "#PWR12" H 2800 5050 50  0001 C CNN
+F 0 "#PWR033" H 2800 5050 50  0001 C CNN
 F 1 "+3.3V" H 2800 5340 50  0000 C CNN
 F 2 "" H 2800 5200 50  0001 C CNN
@@
 Connection ~ 2600 5700
 $Comp
-L GND #PWR6
+L GND #PWR034
 U 1 1 5B8D9B8B
 P 1600 5100
-F 0 "#PWR6" H 1600 4850 50  0001 C CNN
+F 0 "#PWR034" H 1600 4850 50  0001 C CNN
 F 1 "GND" H 1600 4950 50  0000 C CNN
 F 2 "" H 1600 5100 50  0001 C CNN
@@
 $EndComp
 $Comp
-L GND #PWR17
+L GND #PWR035
 U 1 1 5B8DAA78
 P 5800 5600
-F 0 "#PWR17" H 5800 5350 50  0001 C CNN
+F 0 "#PWR035" H 5800 5350 50  0001 C CNN
 F 1 "GND" H 5800 5450 50  0000 C CNN
 F 2 "" H 5800 5600 50  0001 C CNN
@@
 $EndComp
 $Comp
-L GND #PWR20
+L GND #PWR036
 U 1 1 5B8DC59B
 P 6000 3900
-F 0 "#PWR20" H 6000 3650 50  0001 C CNN
+F 0 "#PWR036" H 6000 3650 50  0001 C CNN
 F 1 "GND" H 6000 3750 50  0000 C CNN
 F 2 "" H 6000 3900 50  0001 C CNN
@@
 $EndComp
 $Comp
-L +3.3V #PWR19
+L +3.3V #PWR037
 U 1 1 5B8DC676
 P 6000 2900
-F 0 "#PWR19" H 6000 2750 50  0001 C CNN
+F 0 "#PWR037" H 6000 2750 50  0001 C CNN
 F 1 "+3.3V" H 6000 3040 50  0000 C CNN
 F 2 "" H 6000 2900 50  0001 C CNN
@@
 	8500 3700 8500 4300
 $Comp
-L PWR_FLAG #FLG4
+L PWR_FLAG #FLG038
 U 1 1 5B8FFB6B
 P 8500 3700
-F 0 "#FLG4" H 8500 3775 50  0001 C CNN
+F 0 "#FLG038" H 8500 3775 50  0001 C CNN
 F 1 "PWR_FLAG" H 8500 3850 50  0000 C CNN
 F 2 "" H 8500 3700 50  0001 C CNN
@@
 $EndComp
 $Comp
-L GND #PWR7
+L GND #PWR039
 U 1 1 5B9D7B32
 P 1650 3450
-F 0 "#PWR7" H 1650 3200 50  0001 C CNN
+F 0 "#PWR039" H 1650 3200 50  0001 C CNN
 F 1 "GND" H 1650 3300 50  0000 C CNN
 F 2 "" H 1650 3450 50  0001 C CNN
@@
 $EndComp
 $Comp
-L GND #PWR36
+L GND #PWR040
 U 1 1 5B9F33CF
 P 9600 4250
-F 0 "#PWR36" H 9600 4000 50  0001 C CNN
+F 0 "#PWR040" H 9600 4000 50  0001 C CNN
 F 1 "GND" H 9600 4100 50  0000 C CNN
 F 2 "" H 9600 4250 50  0001 C CNN
@@
 $EndComp
 $Comp
-L GND #PWR28
+L GND #PWR041
 U 1 1 5B9F3B03
 P 7550 4300
-F 0 "#PWR28" H 7550 4050 50  0001 C CNN
+F 0 "#PWR041" H 7550 4050 50  0001 C CNN
 F 1 "GND" H 7550 4150 50  0000 C CNN
 F 2 "" H 7550 4300 50  0001 C CNN
@@
 	7550 4000 7550 3900
 Connection ~ 7550 3900
+Text Label 7700 2200 0    60   ~ 0
+B1-A
+Text Label 7700 2500 0    60   ~ 0
+B1-B
 $EndSCHEMATC
