File: kicad/uc2.sch (KiCad schematic (older format))
At the start: 75 parts, among them J17 PRJ_USB_MINI, J18 Conn_01x05, J19 SOLDERBRDIGE-3, J20 Conn_01x05, J21 SOLDERBRDIGE-3, J22 SOLDERBRDIGE-2, J23 UART-Harwin3, J24 Conn_02x03_Odd_Even, J25 Atmega-ISP-6, J26 Conn_01x03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

Commit message: PCB V0.1 Tapeout
Connections:
- net B3-A: now reaches J26.2 (Pin_2), R32.2, U6.6 (A)
- net B3-B: now reaches J26.3 (Pin_3), R33.2, U6.7 (B)
- net B2-A: now reaches J27.2 (Pin_2), R34.2, U7.6 (A)
- net B2-B: now reaches J27.3 (Pin_3), R35.2, U7.7 (B)
Changed lines of the file:
@@
 $EndDescr
 $Comp
-L +3.3V #PWR50
+L +3.3V #PWR042
 U 1 1 5B8EEC2D
 P 3700 700
-F 0 "#PWR50" H 3700 550 50  0001 C CNN
+F 0 "#PWR042" H 3700 550 50  0001 C CNN
 F 1 "+3.3V" H 3700 840 50  0000 C CNN
 F 2 "" H 3700 700 50  0001 C CNN
@@
 $EndComp
 $Comp
-L GND #PWR51
+L GND #PWR043
 U 1 1 5B8EEC33
 P 3700 5700
-F 0 "#PWR51" H 3700 5450 50  0001 C CNN
+F 0 "#PWR043" H 3700 5450 50  0001 C CNN
 F 1 "GND" H 3700 5550 50  0000 C CNN
 F 2 "" H 3700 5700 50  0001 C CNN
@@
 $EndComp
 $Comp
-L GND #PWR52
+L GND #PWR044
 U 1 1 5B8EEC5F
 P 4800 1300
-F 0 "#PWR52" H 4800 1050 50  0001 C CNN
+F 0 "#PWR044" H 4800 1050 50  0001 C CNN
 F 1 "GND" H 4800 1150 50  0000 C CNN
 F 2 "" H 4800 1300 50  0001 C CNN
@@
 $EndComp
 $Comp
-L GND #PWR47
+L GND #PWR045
 U 1 1 5B8EEC6C
 P 2800 3400
-F 0 "#PWR47" H 2800 3150 50  0001 C CNN
+F 0 "#PWR045" H 2800 3150 50  0001 C CNN
 F 1 "GND" H 2800 3250 50  0000 C CNN
 F 2 "" H 2800 3400 50  0001 C CNN
@@
 $EndComp
 $Comp
-L GND #PWR44
+L GND #PWR046
 U 1 1 5B8EEC82
 P 1900 2700
-F 0 "#PWR44" H 1900 2450 50  0001 C CNN
+F 0 "#PWR046" H 1900 2450 50  0001 C CNN
 F 1 "GND" H 1900 2550 50  0000 C CNN
 F 2 "" H 1900 2700 50  0001 C CNN
@@
 $EndComp
 $Comp
-L +3.3V #PWR45
+L +3.3V #PWR047
 U 1 1 5B8EECDB
 P 2300 700
-F 0 "#PWR45" H 2300 550 50  0001 C CNN
+F 0 "#PWR047" H 2300 550 50  0001 C CNN
 F 1 "+3.3V" H 2300 840 50  0000 C CNN
 F 2 "" H 2300 700 50  0001 C CNN
@@
 $EndComp
 $Comp
-L GND #PWR41
+L GND #PWR048
 U 1 1 5B8EECE1
 P 1600 1900
-F 0 "#PWR41" H 1600 1650 50  0001 C CNN
+F 0 "#PWR048" H 1600 1650 50  0001 C CNN
 F 1 "GND" H 1600 1750 50  0000 C CNN
 F 2 "" H 1600 1900 50  0001 C CNN
@@
 $EndComp
 $Comp
-L +3.3V #PWR70
+L +3.3V #PWR049
 U 1 1 5B8EED52
 P 9100 1100
-F 0 "#PWR70" H 9100 950 50  0001 C CNN
+F 0 "#PWR049" H 9100 950 50  0001 C CNN
 F 1 "+3.3V" H 9100 1240 50  0000 C CNN
 F 2 "" H 9100 1100 50  0001 C CNN
@@
 $EndComp
 $Comp
-L GND #PWR74
+L GND #PWR050
 U 1 1 5B8EED60
 P 10100 2100
-F 0 "#PWR74" H 10100 1850 50  0001 C CNN
+F 0 "#PWR050" H 10100 1850 50  0001 C CNN
 F 1 "GND" H 10100 1950 50  0000 C CNN
 F 2 "" H 10100 2100 50  0001 C CNN
@@
 $EndComp
 $Comp
-L GND #PWR71
+L GND #PWR051
 U 1 1 5B8EED92
 P 9100 2900
-F 0 "#PWR71" H 9100 2650 50  0001 C CNN
+F 0 "#PWR051" H 9100 2650 50  0001 C CNN
 F 1 "GND" H 9100 2750 50  0000 C CNN
 F 2 "" H 9100 2900 50  0001 C CNN
@@
 $EndComp
 $Comp
-L GND #PWR66
+L GND #PWR052
 U 1 1 5B8EEDAE
 P 7900 1400
-F 0 "#PWR66" H 7900 1150 50  0001 C CNN
+F 0 "#PWR052" H 7900 1150 50  0001 C CNN
 F 1 "GND" H 7900 1250 50  0000 C CNN
 F 2 "" H 7900 1400 50  0001 C CNN
@@
 $EndComp
 $Comp
-L GND #PWR59
+L GND #PWR053
 U 1 1 5B8EEDC2
 P 6600 2800
-F 0 "#PWR59" H 6600 2550 50  0001 C CNN
+F 0 "#PWR053" H 6600 2550 50  0001 C CNN
 F 1 "GND" H 6600 2650 50  0000 C CNN
 F 2 "" H 6600 2800 50  0001 C CNN
@@
 $EndComp
 $Comp
-L +3.3V #PWR58
+L +3.3V #PWR054
 U 1 1 5B8EEDDD
 P 6600 1200
-F 0 "#PWR58" H 6600 1050 50  0001 C CNN
+F 0 "#PWR054" H 6600 1050 50  0001 C CNN
 F 1 "+3.3V" H 6600 1340 50  0000 C CNN
 F 2 "" H 6600 1200 50  0001 C CNN
@@
 $EndComp
 $Comp
-L +3.3V #PWR54
+L +3.3V #PWR055
 U 1 1 5B8EEDF6
 P 6000 800
-F 0 "#PWR54" H 6000 650 50  0001 C CNN
+F 0 "#PWR055" H 6000 650 50  0001 C CNN
 F 1 "+3.3V" H 6000 940 50  0000 C CNN
 F 2 "" H 6000 800 50  0001 C CNN
@@
 $EndComp
 $Comp
-L +3.3V #PWR62
+L +3.3V #PWR056
 U 1 1 5B8EEE07
 P 7400 1100
-F 0 "#PWR62" H 7400 950 50  0001 C CNN
+F 0 "#PWR056" H 7400 950 50  0001 C CNN
 F 1 "+3.3V" H 7400 1240 50  0000 C CNN
 F 2 "" H 7400 1100 50  0001 C CNN
@@
 $EndComp
 $Comp
-L GND #PWR63
+L GND #PWR057
 U 1 1 5B8EEE19
 P 7400 2700
-F 0 "#PWR63" H 7400 2450 50  0001 C CNN
+F 0 "#PWR057" H 7400 2450 50  0001 C CNN
 F 1 "GND" H 7400 2550 50  0000 C CNN
 F 2 "" H 7400 2700 50  0001 C CNN
@@
 $EndComp
 $Comp
-L GND #PWR46
+L GND #PWR058
 U 1 1 5B8EEE27
 P 2300 7450
-F 0 "#PWR46" H 2300 7200 50  0001 C CNN
+F 0 "#PWR058" H 2300 7200 50  0001 C CNN
 F 1 "GND" H 2300 7300 50  0000 C CNN
 F 2 "" H 2300 7450 50  0001 C CNN
@@
 $EndComp
 $Comp
-L GND #PWR40
+L GND #PWR059
 U 1 1 5B8EEE2D
 P 1500 7000
-F 0 "#PWR40" H 1500 6750 50  0001 C CNN
+F 0 "#PWR059" H 1500 6750 50  0001 C CNN
 F 1 "GND" H 1500 6850 50  0000 C CNN
 F 2 "" H 1500 7000 50  0001 C CNN
@@
 NoConn ~ 2800 6600
 $Comp
-L +3.3V #PWR48
+L +3.3V #PWR060
 U 1 1 5B8EEE3E
 P 2900 5200
-F 0 "#PWR48" H 2900 5050 50  0001 C CNN
+F 0 "#PWR060" H 2900 5050 50  0001 C CNN
 F 1 "+3.3V" H 2900 5340 50  0000 C CNN
 F 2 "" H 2900 5200 50  0001 C CNN
@@
 $EndComp
 $Comp
-L GND #PWR38
+L GND #PWR061
 U 1 1 5B8EEE54
 P 900 6900
-F 0 "#PWR38" H 900 6650 50  0001 C CNN
+F 0 "#PWR061" H 900 6650 50  0001 C CNN
 F 1 "GND" H 900 6750 50  0000 C CNN
 F 2 "" H 900 6900 50  0001 C CNN
@@
 $EndComp
 $Comp
-L GND #PWR43
+L GND #PWR062
 U 1 1 5B8EEE63
 P 1800 5900
-F 0 "#PWR43" H 1800 5650 50  0001 C CNN
+F 0 "#PWR062" H 1800 5650 50  0001 C CNN
 F 1 "GND" H 1800 5750 50  0000 C CNN
 F 2 "" H 1800 5900 50  0001 C CNN
@@
 UC2-MOSI
 $Comp
-L GND #PWR69
+L GND #PWR063
 U 1 1 5B8EEE7E
 P 8700 6200
-F 0 "#PWR69" H 8700 5950 50  0001 C CNN
+F 0 "#PWR063" H 8700 5950 50  0001 C CNN
 F 1 "GND" H 8700 6050 50  0000 C CNN
 F 2 "" H 8700 6200 50  0001 C CNN
@@
 $EndComp
 $Comp
-L +3.3V #PWR68
+L +3.3V #PWR064
 U 1 1 5B8EEE86
 P 8700 5600
-F 0 "#PWR68" H 8700 5450 50  0001 C CNN
+F 0 "#PWR064" H 8700 5450 50  0001 C CNN
 F 1 "+3.3V" H 8700 5740 50  0000 C CNN
 F 2 "" H 8700 5600 50  0001 C CNN
@@
 $EndComp
 $Comp
-L +3.3V #PWR57
+L +3.3V #PWR065
 U 1 1 5B8EEED6
 P 6200 5000
-F 0 "#PWR57" H 6200 4850 50  0001 C CNN
+F 0 "#PWR065" H 6200 4850 50  0001 C CNN
 F 1 "+3.3V" H 6200 5140 50  0000 C CNN
 F 2 "" H 6200 5000 50  0001 C CNN
@@
 $EndComp
 $Comp
-L +3.3V #PWR72
+L +3.3V #PWR066
 U 1 1 5B8F7DB6
 P 9100 3400
-F 0 "#PWR72" H 9100 3250 50  0001 C CNN
+F 0 "#PWR066" H 9100 3250 50  0001 C CNN
 F 1 "+3.3V" H 9100 3540 50  0000 C CNN
 F 2 "" H 9100 3400 50  0001 C CNN
@@
 $EndComp
 $Comp
-L GND #PWR75
+L GND #PWR067
 U 1 1 5B8F7DCA
 P 10100 4400
-F 0 "#PWR75" H 10100 4150 50  0001 C CNN
+F 0 "#PWR067" H 10100 4150 50  0001 C CNN
 F 1 "GND" H 10100 4250 50  0000 C CNN
 F 2 "" H 10100 4400 50  0001 C CNN
@@
 $EndComp
 $Comp
-L GND #PWR73
+L GND #PWR068
 U 1 1 5B8F7DF8
 P 9100 5200
-F 0 "#PWR73" H 9100 4950 50  0001 C CNN
+F 0 "#PWR068" H 9100 4950 50  0001 C CNN
 F 1 "GND" H 9100 5050 50  0000 C CNN
 F 2 "" H 9100 5200 50  0001 C CNN
@@
 $EndComp
 $Comp
-L GND #PWR67
+L GND #PWR069
 U 1 1 5B8F7E15
 P 7900 3700
-F 0 "#PWR67" H 7900 3450 50  0001 C CNN
+F 0 "#PWR069" H 7900 3450 50  0001 C CNN
 F 1 "GND" H 7900 3550 50  0000 C CNN
 F 2 "" H 7900 3700 50  0001 C CNN
@@
 $EndComp
 $Comp
-L GND #PWR61
+L GND #PWR070
 U 1 1 5B8F7E2D
 P 6800 5100
-F 0 "#PWR61" H 6800 4850 50  0001 C CNN
+F 0 "#PWR070" H 6800 4850 50  0001 C CNN
 F 1 "GND" H 6800 4950 50  0000 C CNN
 F 2 "" H 6800 5100 50  0001 C CNN
@@
 $EndComp
 $Comp
-L +3.3V #PWR56
+L +3.3V #PWR071
 U 1 1 5B8F7E48
 P 6200 3500
-F 0 "#PWR56" H 6200 3350 50  0001 C CNN
+F 0 "#PWR071" H 6200 3350 50  0001 C CNN
 F 1 "+3.3V" H 6200 3640 50  0000 C CNN
 F 2 "" H 6200 3500 50  0001 C CNN
@@
 $EndComp
 $Comp
-L +3.3V #PWR64
+L +3.3V #PWR072
 U 1 1 5B8F7E54
 P 7400 3400
-F 0 "#PWR64" H 7400 3250 50  0001 C CNN
+F 0 "#PWR072" H 7400 3250 50  0001 C CNN
 F 1 "+3.3V" H 7400 3540 50  0000 C CNN
 F 2 "" H 7400 3400 50  0001 C CNN
@@
 $EndComp
 $Comp
-L GND #PWR65
+L GND #PWR073
 U 1 1 5B8F7E67
 P 7400 5000
-F 0 "#PWR65" H 7400 4750 50  0001 C CNN
+F 0 "#PWR073" H 7400 4750 50  0001 C CNN
 F 1 "GND" H 7400 4850 50  0000 C CNN
 F 2 "" H 7400 5000 50  0001 C CNN
@@
 NoConn ~ 5000 2700
 $Comp
-L GND #PWR55
+L GND #PWR074
 U 1 1 5B9025AE
 P 6050 2800
-F 0 "#PWR55" H 6050 2550 50  0001 C CNN
+F 0 "#PWR074" H 6050 2550 50  0001 C CNN
 F 1 "GND" H 6050 2650 50  0000 C CNN
 F 2 "" H 6050 2800 50  0001 C CNN
@@
 $EndComp
 $Comp
-L GND #PWR53
+L GND #PWR075
 U 1 1 5B8EB6F2
 P 5400 7100
-F 0 "#PWR53" H 5400 6850 50  0001 C CNN
+F 0 "#PWR075" H 5400 6850 50  0001 C CNN
 F 1 "GND" H 5400 6950 50  0000 C CNN
 F 2 "" H 5400 7100 50  0001 C CNN
@@
 $EndComp
 $Comp
-L PWR_FLAG #FLG5
+L PWR_FLAG #FLG076
 U 1 1 5B8FFFC2
 P 2300 5200
-F 0 "#FLG5" H 2300 5275 50  0001 C CNN
+F 0 "#FLG076" H 2300 5275 50  0001 C CNN
 F 1 "PWR_FLAG" H 2300 5350 50  0000 C CNN
 F 2 "" H 2300 5200 50  0001 C CNN
@@
 $EndComp
 $Comp
-L +3.3V #PWR60
+L +3.3V #PWR077
 U 1 1 5B9065EF
 P 6800 3200
-F 0 "#PWR60" H 6800 3050 50  0001 C CNN
+F 0 "#PWR077" H 6800 3050 50  0001 C CNN
 F 1 "+3.3V" H 6800 3340 50  0000 C CNN
 F 2 "" H 6800 3200 50  0001 C CNN
@@
 $EndComp
 $Comp
-L GND #PWR39
+L GND #PWR078
 U 1 1 5B9D84AC
 P 1500 3250
-F 0 "#PWR39" H 1500 3000 50  0001 C CNN
+F 0 "#PWR078" H 1500 3000 50  0001 C CNN
 F 1 "GND" H 1500 3100 50  0000 C CNN
 F 2 "" H 1500 3250 50  0001 C CNN
@@
 $EndComp
 $Comp
-L GND #PWR49
+L GND #PWR079
 U 1 1 5B9F4880
 P 3400 5900
-F 0 "#PWR49" H 3400 5650 50  0001 C CNN
+F 0 "#PWR079" H 3400 5650 50  0001 C CNN
 F 1 "GND" H 3400 5750 50  0000 C CNN
 F 2 "" H 3400 5900 50  0001 C CNN
@@
 $EndComp
 $Comp
-L GND #PWR42
+L GND #PWR080
 U 1 1 5B9F508D
 P 1800 5500
-F 0 "#PWR42" H 1800 5250 50  0001 C CNN
+F 0 "#PWR080" H 1800 5250 50  0001 C CNN
 F 1 "GND" H 1800 5350 50  0000 C CNN
 F 2 "" H 1800 5500 50  0001 C CNN
@@
 Wire Wire Line
 	1800 5500 1800 5400
+Text Label 7800 1900 0    60   ~ 0
+B3-A
+Text Label 7800 2200 0    60   ~ 0
+B3-B
+Text Label 7800 4200 0    60   ~ 0
+B2-A
+Text Label 7800 4500 0    60   ~ 0
+B2-B
 $EndSCHEMATC
